Commit message: migrated our panda_moveit_config to this noetic branch

File: config/hand.xacro (robot description, xacro)
@@ -1,5 +1,5 @@
 <?xml version="1.0" encoding="UTF-8"?>
 <robot xmlns:xacro="http://www.ros.org/wiki/xacro" name="panda">
-    <xacro:macro name="hand">
+    <xacro:macro name="hand" params="gripper_center:='true'">
         <!--GROUPS: Representation of a set of joints and links. This can be useful for specifying DOF to plan for, defining arms, end effectors, etc-->
         <!--LINKS: When a link is specified, the parent joint of that link (if it exists) is automatically included-->
@@ -11,4 +11,8 @@
             <link name="panda_leftfinger"/>
             <link name="panda_rightfinger"/>
+            <!-- Added extra virtual joint to ease the grasp movement planning -->
+            <xacro:if value="${gripper_center}" > <!-- Only when gripper_center==True -->
+                <link name="panda_gripper_center" />
+            </xacro:if>
         </group>
         <!--GROUP STATES: Purpose: Define a named state for a particular group, in terms of joint values. This is useful to define states like 'folded arms'-->
@@ -44,4 +48,5 @@
         <disable_collisions link1="panda_link7" link2="panda_rightfinger" reason="Never"/>
         <disable_collisions link1="panda_link8" link2="panda_rightfinger" reason="Never"/>
+        <disable_collisions link1="panda_hand" link2="camera_arm_link" reason="Adjacent"/>
     </xacro:macro>
 </robot>

File: config/panda.srdf.xacro (robot description, xacro)
@@ -5,13 +5,29 @@
 -->
 <robot xmlns:xacro="http://www.ros.org/wiki/xacro" name="panda">
+    <!-- Initialize gripper_center properties -->
+    <xacro:arg name="gripper_center" default="true" />
+    <xacro:property name="gripper_center" value="$(arg gripper_center)"/>
+    <!-- Initialize on_mobile_base properties -->
+    <xacro:arg name="on_mobile_base" default="true" />
+    <xacro:property name="on_mobile_base" value="$(arg on_mobile_base)"/>
     <xacro:include filename="$(find panda_moveit_config)/config/panda_arm.xacro" />
-    <xacro:panda_arm />
-    <xacro:arg name="hand" default="false" />
+    <xacro:panda_arm on_mobile_base="${on_mobile_base}"/>
+    <xacro:arg name="hand" default="true" />
     <!--Add the hand if people request it-->
     <xacro:if value="$(arg hand)">
         <xacro:include filename="$(find panda_moveit_config)/config/hand.xacro" />
-        <xacro:hand />
+        <xacro:hand gripper_center="${gripper_center}" /> <!-- Added extra xacro macro argument for the new virtual center gripper link -->/>
+        <group name="panda_arm_hand">
+            <group name="panda_arm" />
+            <group name="hand" />
+        </group>
         <!--END EFFECTOR: Purpose: Represent information about an end effector.-->
-        <end_effector name="hand" parent_link="panda_link8" group="hand"/>
+        <!--END EFFECTOR: Purpose: Represent information about an end effector.-->
+        <!--end_effector name="hand" parent_link="panda_link8" group="hand" parent_group="panda_arm" / -->
+        <!-- Added extra virtual joint to ease the grasp movement planning -->
+        <!-- xacro:if value="${gripper_center}" --> <!-- Only when gripper_center==True -->
+        <!-- virtual_joint name="world" type="planar" parent_frame="world" child_link="panda_link0" /-->
+        <end_effector name="gripper_center" parent_link="panda_gripper_center" group="hand" parent_group="panda_arm" />
+        <!-- /xacro:if -->
     </xacro:if>
 </robot>

File: config/panda_arm.xacro (robot description, xacro)
@@ -1,60 +1,228 @@
 <?xml version="1.0" encoding="UTF-8"?>
 <robot xmlns:xacro="http://www.ros.org/wiki/xacro" name="panda">
-    <xacro:macro name="panda_arm">
-        <!--GROUPS: Representation of a set of joints and links. This can be useful for specifying DOF to plan for, defining arms, end effectors, etc-->
-        <!--LINKS: When a link is specified, the parent joint of that link (if it exists) is automatically included-->
-        <!--JOINTS: When a joint is specified, the child link of that joint (which will always exist) is automatically included-->
-        <!--CHAINS: When a chain is specified, all the links along the chain (including endpoints) are included in the group. Additionally, all the joints that are parents to included links are also included. This means that joints along the chain and the parent joint of the base link are included in the group-->
-        <!--SUBGROUPS: Groups can also be formed by referencing to already defined group names-->
-        <group name="panda_arm">
-            <chain base_link="panda_link0" tip_link="panda_link8"/>
-        </group>
-        <!--GROUP STATES: Purpose: Define a named state for a particular group, in terms of joint values. This is useful to define states like 'folded arms'-->
-        <group_state name="ready" group="panda_arm">
-            <joint name="panda_joint1" value="0"/>
-            <joint name="panda_joint2" value="-0.785"/>
-            <joint name="panda_joint3" value="0"/>
-            <joint name="panda_joint4" value="-2.356"/>
-            <joint name="panda_joint5" value="0"/>
-            <joint name="panda_joint6" value="1.571"/>
-            <joint name="panda_joint7" value="-0.7855"/>
-        </group_state>
-        <group_state name="extended" group="panda_arm">
-            <joint name="panda_joint1" value="0"/>
-            <joint name="panda_joint2" value="-0.3927"/>
-            <joint name="panda_joint3" value="0"/>
-            <joint name="panda_joint4" value="-0.7855"/>
-            <joint name="panda_joint5" value="0"/>
-            <joint name="panda_joint6" value="3.142"/>
-            <joint name="panda_joint7" value="-0.785"/>
-        </group_state>
-        <!--VIRTUAL JOINT: Purpose: this element defines a virtual joint between a robot link and an external frame of reference (considered fixed with respect to the robot)-->
-        <virtual_joint name="virtual_joint" type="fixed" parent_frame="world" child_link="panda_link0"/>
-        <!--DISABLE COLLISIONS: By default it is assumed that any link of the robot could potentially come into collision with any other link in the robot. This tag disables collision checking between a specified pair of links. -->
-        <disable_collisions link1="panda_link0" link2="panda_link1" reason="Adjacent"/>
-        <disable_collisions link1="panda_link0" link2="panda_link2" reason="Never"/>
-        <disable_collisions link1="panda_link0" link2="panda_link3" reason="Never"/>
-        <disable_collisions link1="panda_link0" link2="panda_link4" reason="Never"/>
-        <disable_collisions link1="panda_link1" link2="panda_link2" reason="Adjacent"/>
-        <disable_collisions link1="panda_link1" link2="panda_link3" reason="Default"/>
-        <disable_collisions link1="panda_link1" link2="panda_link4" reason="Never"/>
-        <disable_collisions link1="panda_link2" link2="panda_link3" reason="Adjacent"/>
-        <disable_collisions link1="panda_link2" link2="panda_link4" reason="Never"/>
-        <disable_collisions link1="panda_link3" link2="panda_link4" reason="Adjacent"/>
-        <disable_collisions link1="panda_link3" link2="panda_link6" reason="Never"/>
-        <disable_collisions link1="panda_link4" link2="panda_link5" reason="Adjacent"/>
-        <disable_collisions link1="panda_link4" link2="panda_link6" reason="Never"/>
-        <disable_collisions link1="panda_link4" link2="panda_link7" reason="Never"/>
-        <disable_collisions link1="panda_link4" link2="panda_link8" reason="Never"/>
-        <disable_collisions link1="panda_link5" link2="panda_link6" reason="Adjacent"/>
-        <disable_collisions link1="panda_link5" link2="panda_link7" reason="Default"/>
-        <disable_collisions link1="panda_link6" link2="panda_link7" reason="Adjacent"/>
-        <disable_collisions link1="panda_link7" link2="panda_link8" reason="Adjacent"/>
-        <!-- Fix self-collisions between too coarse collision geometries provided by franka_description
-             See https://github.com/ros-planning/panda_moveit_config/issues/72#issuecomment-768472329
-                 https://github.com/ros-planning/panda_moveit_config/pull/35#pullrequestreview-390715967
-        -->
-        <disable_collisions link1="panda_link5" link2="panda_link8" reason="Default" />
-        <disable_collisions link1="panda_link6" link2="panda_link8" reason="Default"/>
-    </xacro:macro>
+  <xacro:macro name="panda_arm" params="on_mobile_base:='true'" >
+    <!--GROUPS: Representation of a set of joints and links. This can be useful for specifying DOF to plan for, defining arms, end effectors, etc-->
+    <!--LINKS: When a link is specified, the parent joint of that link (if it exists) is automatically included-->
+    <!--JOINTS: When a joint is specified, the child link of that joint (which will always exist) is automatically included-->
+    <!--CHAINS: When a chain is specified, all the links along the chain (including endpoints) are included in the group. Additionally, all the joints that are parents to included links are also included. This means that joints along the chain and the parent joint of the base link are included in the group-->
+    <!--SUBGROUPS: Groups can also be formed by referencing to already defined group names-->
+    <group name="panda_arm">
+      <link name="panda_gripper_center" />
+      <joint name="panda_joint1" />
+      <joint name="panda_joint2" />
+      <joint name="panda_joint3" />
+      <joint name="panda_joint4" />
+      <joint name="panda_joint5" />
+      <joint name="panda_joint6" />
+      <joint name="panda_joint7" />
+      <joint name="panda_joint8" />
+      <chain base_link="panda_link0" tip_link="panda_link8" />
+    </group>
+    <!--GROUP STATES: Purpose: Define a named state for a particular group, in terms of joint values. This is useful to define states like 'folded arms'-->
+    <group_state name="ready" group="panda_arm">
+      <joint name="panda_joint1" value="0" />
+      <joint name="panda_joint2" value="-0.785" />
+      <joint name="panda_joint3" value="0" />
+      <joint name="panda_joint4" value="-2.356" />
+      <joint name="panda_joint5" value="0" />
+      <joint name="panda_joint6" value="1.571" />
+      <joint name="panda_joint7" value="0.785" />
+    </group_state>
+    <group_state name="ahead" group="panda_arm">
+      <joint name="panda_joint1" value="0" />
+      <joint name="panda_joint2" value="-0.959" />
+      <joint name="panda_joint3" value="0" />
+      <joint name="panda_joint4" value="-2.356" />
+      <joint name="panda_joint5" value="0" />
+      <joint name="panda_joint6" value="2.967" />
+      <joint name="panda_joint7" value="0.785" />
+    </group_state>
+    <group_state name="extended" group="panda_arm">
+      <joint name="panda_joint1" value="0" />
+      <joint name="panda_joint2" value="0" />
+      <joint name="panda_joint3" value="0" />
+      <joint name="panda_joint4" value="-0.0698" />
+      <joint name="panda_joint5" value="0" />
+      <joint name="panda_joint6" value="0.5" />
+      <joint name="panda_joint7" value="0.785" />
+    </group_state>
+    <group_state name="transport" group="panda_arm">
+      <joint name="panda_joint1" value="0" />
+      <joint name="panda_joint2" value="-0.5599" />
+      <joint name="panda_joint3" value="0" />
+      <joint name="panda_joint4" value="-2.97" />
+      <joint name="panda_joint5" value="0" />
+      <joint name="panda_joint6" value="0" />
+      <joint name="panda_joint7" value="0.785" />
+    </group_state>
+<!--
+rosservice call /franka_move_node/move_joints "{joint_1: 0.0, joint_2: -1.5, joint_3: 0.0, joint_4: -3.5, joint_5: 0.0, joint_6: 1.57,
+  joint_7: 0.79}" -->
+    <group_state name="drive" group="panda_arm">
+      <joint name="panda_joint1" value="0" />
+      <joint name="panda_joint2" value="-1.65" />
+      <joint name="panda_joint3" value="0" />
+      <joint name="panda_joint4" value="-2.9" />
+      <joint name="panda_joint5" value="0" />
+      <joint name="panda_joint6" value="2.5" />
+      <joint name="panda_joint7" value="0.785" />
+    </group_state>
+    <group_state name="poseDeskFront" group="panda_arm">
+      <joint name="panda_joint1" value="0.0" />
+      <joint name="panda_joint2" value="-0.2" />
+      <joint name="panda_joint3" value="0.0" />
+      <joint name="panda_joint4" value="-1.8" />
+      <joint name="panda_joint5" value="0.0" />
+      <joint name="panda_joint6" value="1.6" />
+      <joint name="panda_joint7" value="0.785" />
+    </group_state>
+    <group_state name="poseDeskLeft" group="panda_arm">
+      <joint name="panda_joint1" value="1.57" />
+      <joint name="panda_joint2" value="0.15" />
+      <joint name="panda_joint3" value="0" />
+      <joint name="panda_joint4" value="-1.4" />
+      <joint name="panda_joint5" value="0" />
+      <joint name="panda_joint6" value="1.6" />
+      <joint name="panda_joint7" value="0.785" />
+    </group_state>
+    <group_state name="poseDeskRight" group="panda_arm">
+      <joint name="panda_joint1" value="-1.57" />
+      <joint name="panda_joint2" value="0.15" />
+      <joint name="panda_joint3" value="0" />
+      <joint name="panda_joint4" value="-1.4" />
+      <joint name="panda_joint5" value="0" />
+      <joint name="panda_joint6" value="1.6" />
+      <joint name="panda_joint7" value="0.785" />
+    </group_state>
+    <group_state name="poseShelfTopFront" group="panda_arm">
+      <joint name="panda_joint1" value="0.0" />
+      <joint name="panda_joint2" value="0" />
+      <joint name="panda_joint3" value="0" />
+      <joint name="panda_joint4" value="-0.0698" />
+      <joint name="panda_joint5" value="0" />
+      <joint name="panda_joint6" value="0.5" />
+      <joint name="panda_joint7" value="0.785" />
+    </group_state>
+    <group_state name="poseShelfTopLeft" group="panda_arm">
+      <joint name="panda_joint1" value="0" />
+      <joint name="panda_joint2" value="0" />
+      <joint name="panda_joint3" value="0" />
+      <joint name="panda_joint4" value="-0.0698" />
+      <joint name="panda_joint5" value="0" />
+      <joint name="panda_joint6" value="0.5" />
+      <joint name="panda_joint7" value="0.785" />
+    </group_state>
+    <group_state name="poseShelfTopRight" group="panda_arm">
+      <joint name="panda_joint1" value="0" />
+      <joint name="panda_joint2" value="0" />
+      <joint name="panda_joint3" value="0" />
+      <joint name="panda_joint4" value="-0.0698" />
+      <joint name="panda_joint5" value="0" />
+      <joint name="panda_joint6" value="0.5" />
+      <joint name="panda_joint7" value="0.785" />
+    </group_state>
+    <group_state name="poseShelfBottomFront" group="panda_arm">
+      <joint name="panda_joint1" value="0.0" />
+      <joint name="panda_joint2" value="-0.2" />
+      <joint name="panda_joint3" value="0.0" />
+      <joint name="panda_joint4" value="-1.8" />
+      <joint name="panda_joint5" value="0.0" />
+      <joint name="panda_joint6" value="1.6" />
+      <joint name="panda_joint7" value="0.785" />
+    </group_state>
+    <group_state name="poseShelfBottomLeft" group="panda_arm">
+      <joint name="panda_joint1" value="1.57" />
+      <joint name="panda_joint2" value="-0.2" />
+      <joint name="panda_joint3" value="0.0" />
+      <joint name="panda_joint4" value="-1.8" />
+      <joint name="panda_joint5" value="0.0" />
+      <joint name="panda_joint6" value="1.6" />
+      <joint name="panda_joint7" value="0.785" />
+    </group_state>
+    <group_state name="poseShelfBottomRight" group="panda_arm">
+      <joint name="panda_joint1" value="-1.57" />
+      <joint name="panda_joint2" value="-0.2" />
+      <joint name="panda_joint3" value="0.0" />
+      <joint name="panda_joint4" value="-1.8" />
+      <joint name="panda_joint5" value="0.0" />
+      <joint name="panda_joint6" value="1.6" />
+      <joint name="panda_joint7" value="0.785" />
+    </group_state>
+    <group_state name="poseTransportPlateLeft" group="panda_arm">
+      <joint name="panda_joint1" value="+2.8" />
+      <joint name="panda_joint2" value="-0.4" />
+      <joint name="panda_joint3" value="0" />
+      <joint name="panda_joint4" value="-2.5" />
+      <joint name="panda_joint5" value="0" />
+      <joint name="panda_joint6" value="2.3" />
+      <joint name="panda_joint7" value="0.785" />
+    </group_state>
+    <group_state name="poseTransportPlateLeftCenter" group="panda_arm">
+      <joint name="panda_joint1" value="-1.6" />
+      <joint name="panda_joint2" value="-1.5" />
+      <joint name="panda_joint3" value="-1.14" />
+      <joint name="panda_joint4" value="-2.19" />
+      <joint name="panda_joint5" value="-1.32" />
+      <joint name="panda_joint6" value="1.3" />
+      <joint name="panda_joint7" value="1.04" />
+    </group_state>
+    <group_state name="poseTransportPlateRight" group="panda_arm">
+      <joint name="panda_joint1" value="-2.8" />
+      <joint name="panda_joint2" value="-0.58" />
+      <joint name="panda_joint3" value="0" />
+      <joint name="panda_joint4" value="-2.8" />
+      <joint name="panda_joint5" value="0" />
+      <joint name="panda_joint6" value="2.3" />
+      <joint name="panda_joint7" value="0.785" />
+    </group_state>
+    <group_state name="poseTransportPlateRightCenter" group="panda_arm">
+      <joint name="panda_joint1" value="1.42" />
+      <joint name="panda_joint2" value="-1.15" />
+      <joint name="panda_joint3" value="0.95" />
+      <joint name="panda_joint4" value="-1.677" />
+      <joint name="panda_joint5" value="1.02" />
+      <joint name="panda_joint6" value="1.06" />
+      <joint name="panda_joint7" value="0.252" />
+    </group_state>
+    <group_state name="poseTransportPlateLeftCenter" group="panda_arm">
+      <joint name="panda_joint1" value="-1.4" />
+      <joint name="panda_joint2" value="0.755" />
+      <joint name="panda_joint3" value="-2.0" />
+      <joint name="panda_joint4" value="-1.727" />
+      <joint name="panda_joint5" value="0.667" />
+      <joint name="panda_joint6" value="1.37" />
+      <joint name="panda_joint7" value="0.484" />
+    </group_state>
+    <!-- The virtual joint is used to set pandas planning frame. This will be the parent_frame. -->
+    <!-- If the type is set to planar it is expected that the panda is mounted on a mobile platform. If the panda is static use type fixed. -->
+    <!--xacro:if value="${on_mobile_base}"-->
+    <virtual_joint name="base_joint_virtual" type="planar" parent_frame="panda_base" child_link="panda_link0" /> <!--xyz="0.211 0.0 0.051" /-->
+    <!--/xacro:if-->
+    <xacro:unless value="${on_mobile_base}">
+      <!--virtual_joint name="base_joint_virtual" type="fixed" parent_frame="panda_base" child_link="panda_link0" /--> <!--xyz="0.211 0.0 0.051" /-->
+    </xacro:unless>
+    <!--END EFFECTOR: Purpose: Represent information about an end effector.-->
+    <!--VIRTUAL JOINT: Purpose: this element defines a virtual joint between a robot link and an external frame of reference (considered fixed with respect to the robot)-->
+    <!-- virtual_joint name="virtual_joint" type="fixed" parent_frame="world" child_link="panda_link0" xyz="0.0 0.0 -0.0512"/ -->
+    <!--DISABLE COLLISIONS: By default it is assumed that any link of the robot could potentially come into collision with any other link in the robot. This tag disables collision checking between a specified pair of links. -->
+    <disable_collisions link1="panda_link0" link2="panda_link1" reason="Adjacent" />
+    <disable_collisions link1="panda_link0" link2="panda_link2" reason="Never" />
+    <disable_collisions link1="panda_link0" link2="panda_link3" reason="Never" />
+    <disable_collisions link1="panda_link0" link2="panda_link4" reason="Never" />
+    <disable_collisions link1="panda_link1" link2="panda_link2" reason="Adjacent" />
+    <disable_collisions link1="panda_link1" link2="panda_link3" reason="Default" />
+    <disable_collisions link1="panda_link1" link2="panda_link4" reason="Never" />
+    <disable_collisions link1="panda_link2" link2="panda_link3" reason="Adjacent" />
+    <disable_collisions link1="panda_link2" link2="panda_link4" reason="Never" />
+    <disable_collisions link1="panda_link3" link2="panda_link4" reason="Adjacent" />
+    <disable_collisions link1="panda_link3" link2="panda_link6" reason="Never" />
+    <disable_collisions link1="panda_link4" link2="panda_link5" reason="Adjacent" />
+    <disable_collisions link1="panda_link4" link2="panda_link6" reason="Never" />
+    <disable_collisions link1="panda_link4" link2="panda_link7" reason="Never" />
+    <disable_collisions link1="panda_link4" link2="panda_link8" reason="Never" />
+    <disable_collisions link1="panda_link5" link2="panda_link6" reason="Adjacent" />
+    <disable_collisions link1="panda_link6" link2="panda_link7" reason="Adjacent" />
+    <disable_collisions link1="panda_link6" link2="panda_link8" reason="Default" />
+    <disable_collisions link1="panda_link7" link2="panda_link8" reason="Adjacent" />
+  </xacro:macro>
 </robot>

Commit message: working params for hand open

File: config/hand.xacro (robot description, xacro)
@@ -18,6 +18,6 @@
         <!--GROUP STATES: Purpose: Define a named state for a particular group, in terms of joint values. This is useful to define states like 'folded arms'-->
         <group_state name="open" group="hand">
-            <joint name="panda_finger_joint1" value="0.04"/>
-            <joint name="panda_finger_joint2" value="0.04"/>
+            <joint name="panda_finger_joint1" value="0.039"/>
+            <joint name="panda_finger_joint2" value="0.039"/>
         </group_state>
         <group_state name="close" group="hand">
