Commit message: updated joint limits, added preposition for chessfield

File: config/panda_arm.xacro (robot description, xacro)
@@ -193,4 +193,13 @@
       <joint name="panda_joint6" value="1.37" />
       <joint name="panda_joint7" value="0.484" />
+    </group_state>
+    <group_state name="poseHomeChessBoard" group="panda_arm">
+      <joint name="panda_joint1" value="0.0" />
+      <joint name="panda_joint2" value="0.136" />
+      <joint name="panda_joint3" value="0.0" />
+      <joint name="panda_joint4" value="-2.001" />
+      <joint name="panda_joint5" value="0.0" />
+      <joint name="panda_joint6" value="2.129" />
+      <joint name="panda_joint7" value="0.785" />
     </group_state>
     <!-- The virtual joint is used to set pandas planning frame. This will be the parent_frame. -->

Commit message: added birthday stack

File: config/panda_arm.xacro (robot description, xacro)
@@ -203,5 +203,14 @@
       <joint name="panda_joint7" value="0.785" />
     </group_state>
-    <!-- The virtual joint is used to set pandas planning frame. This will be the parent_frame. -->
+     <group_state name="birthdayStack" group="panda_arm">
+      <joint name="panda_joint1" value="-2.453" />
+      <joint name="panda_joint2" value="-0.259" />
+      <joint name="panda_joint3" value="-0.5392" />
+      <joint name="panda_joint4" value="-1.521" />
+      <joint name="panda_joint5" value="-0.0862" />
+      <joint name="panda_joint6" value="1.3122" />
+      <joint name="panda_joint7" value="0.82" />
+    </group_state>
+   <!-- The virtual joint is used to set pandas planning frame. This will be the parent_frame. -->
     <!-- If the type is set to planar it is expected that the panda is mounted on a mobile platform. If the panda is static use type fixed. -->
     <!--xacro:if value="${on_mobile_base}"-->

Commit message: updated drive joint configuration

File: config/panda_arm.xacro (robot description, xacro)
@@ -61,9 +61,9 @@
     <group_state name="drive" group="panda_arm">
       <joint name="panda_joint1" value="0" />
-      <joint name="panda_joint2" value="-1.65" />
-      <joint name="panda_joint3" value="0" />
-      <joint name="panda_joint4" value="-2.9" />
-      <joint name="panda_joint5" value="0" />
-      <joint name="panda_joint6" value="2.5" />
+      <joint name="panda_joint2" value="-1.45" />
+      <joint name="panda_joint3" value="0" />
+      <joint name="panda_joint4" value="-2.8996" />
+      <joint name="panda_joint5" value="0" />
+      <joint name="panda_joint6" value="1.5" />
       <joint name="panda_joint7" value="0.785" />
     </group_state>
@@ -203,5 +203,5 @@
       <joint name="panda_joint7" value="0.785" />
     </group_state>
-     <group_state name="birthdayStack" group="panda_arm">
+    <group_state name="birthdayStack" group="panda_arm">
       <joint name="panda_joint1" value="-2.453" />
       <joint name="panda_joint2" value="-0.259" />

Commit message: adjusted drive position

File: config/panda_arm.xacro (robot description, xacro)
@@ -61,5 +61,5 @@
     <group_state name="drive" group="panda_arm">
       <joint name="panda_joint1" value="0" />
-      <joint name="panda_joint2" value="-1.65" />
+      <joint name="panda_joint2" value="-1.35" />
       <joint name="panda_joint3" value="0" />
       <joint name="panda_joint4" value="-2.9" />
